File: max20499_breakout.kicad_sch (KiCad schematic)
At the start: 32 parts, among them J1 Conn_01x01, J2 Conn_01x01, J3 Conn_01x04, J4 Conn_01x01, J5 Conn_01x01, U1 MAX20499

Commit message: added manufacturing files, BOM and gerbers.
Parts:
- J1, J2, J4, J5: DK (none) -> A100886CT-ND
Other:
- moved on the sheet: J2
Changed lines of the file:
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@@
     (stroke (width 0) (type default) (color 0 0 0 0))
   )
-  (wire (pts (xy 48.26 76.2) (xy 36.83 76.2))
+  (wire (pts (xy 48.26 76.2) (xy 36.195 76.2))
     (stroke (width 0) (type default) (color 0 0 0 0))
   )
@@
     (pin "2")
   )
-  (symbol (lib_id "Connector_Generic:Conn_01x01") (at 31.75 76.2 180) (unit 1)
+  (symbol (lib_id "Connector_Generic:Conn_01x01") (at 31.115 76.2 180) (unit 1)
     (in_bom yes) (on_board yes)
-    (property "Reference" "J2" (id 0) (at 31.75 73.66 0))
-    (property "Value" "Conn_01x01" (id 1) (at 31.75 71.755 0)
-      (effects (font (size 1.27 1.27)) hide)
-    )
-    (property "Footprint" "low_voltage_reg:63862-1" (id 2) (at 31.75 76.2 0)
-      (effects (font (size 1.27 1.27)) hide)
-    )
-    (property "Datasheet" "~" (id 3) (at 31.75 76.2 0)
+    (property "Reference" "J2" (id 0) (at 31.115 73.66 0))
+    (property "Value" "Conn_01x01" (id 1) (at 31.115 71.755 0)
+      (effects (font (size 1.27 1.27)) hide)
+    )
+    (property "Footprint" "low_voltage_reg:63862-1" (id 2) (at 31.115 76.2 0)
+      (effects (font (size 1.27 1.27)) hide)
+    )
+    (property "Datasheet" "~" (id 3) (at 31.115 76.2 0)
+      (effects (font (size 1.27 1.27)) hide)
+    )
+    (property "DK" "A100886CT-ND" (id 4) (at 31.115 76.2 0)
       (effects (font (size 1.27 1.27)) hide)
     )
@@
       (effects (font (size 1.27 1.27)) hide)
     )
+    (property "DK" "A100886CT-ND" (id 4) (at 31.115 86.995 0)
+      (effects (font (size 1.27 1.27)) hide)
+    )
     (pin "1")
   )
@@
       (effects (font (size 1.27 1.27)) hide)
     )
+    (property "DK" "A100886CT-ND" (id 4) (at 272.415 105.41 0)
+      (effects (font (size 1.27 1.27)) hide)
+    )
     (pin "1")
   )
@@
       (effects (font (size 1.27 1.27)) hide)
     )
+    (property "DK" "A100886CT-ND" (id 4) (at 272.415 94.615 0)
+      (effects (font (size 1.27 1.27)) hide)
+    )
